Commit message: Gazebo fixes: add interia, joint mimics, new name for state publisher package

File: robotiq_2f_85_gripper_visualization/urdf/robotiq_arg2f_85_model_macro.xacro (robot description, xacro)
@@ -4,9 +4,9 @@
   <xacro:macro name="outer_knuckle" params="prefix fingerprefix stroke">
     <link name="${prefix}${fingerprefix}_outer_knuckle">
-      <!--<inertial>
+      <inertial>
         <origin xyz="-0.000200000000003065 0.0199435877845359 0.0292245259211331" rpy="0 0 0" />
         <mass value="0.00853198276973456" />
         <inertia ixx="2.89328108496468E-06" ixy="-1.57935047237397E-19" ixz="-1.93980378593255E-19" iyy="1.86719750325683E-06" iyz="-1.21858577871576E-06" izz="1.21905238907251E-06" />
-        </inertial> -->
+      </inertial>
       <visual>
         <origin xyz="0 0 0" rpy="0 0 0" />
@@ -28,9 +28,9 @@
   <xacro:macro name="outer_finger" params="prefix fingerprefix stroke">
     <link name="${prefix}${fingerprefix}_outer_finger">
-      <!--<inertial>
+      <inertial>
         <origin xyz="0.00030115855001899 0.0373907951953854 -0.0208027427000385" rpy="0 0 0" />
         <mass value="0.022614240507152" />
         <inertia ixx="1.52518312458174E-05" ixy="9.76583423954399E-10" ixz="-5.43838577022588E-10" iyy="6.17694243867776E-06" iyz="6.78636130740228E-06" izz="1.16494917907219E-05" />
-        </inertial> -->
+      </inertial>
       <visual>
         <origin xyz="0 0 0" rpy="0 0 0" />
@@ -52,9 +52,9 @@
   <xacro:macro name="inner_knuckle" params="prefix fingerprefix stroke">
     <link name="${prefix}${fingerprefix}_inner_knuckle">
-      <!--<inertial>
+      <inertial>
         <origin xyz="0.000123011831763771 0.0507850843201817 0.00103968640075166" rpy="0 0 0" />
-       <mass value="0.0271177346495152" />
+        <mass value="0.0271177346495152" />
         <inertia ixx="2.61910379223783E-05" ixy="-2.43616858946494E-07" ixz="-6.37789906117123E-09" iyy="2.8270243746167E-06" iyz="-5.37200748039765E-07" izz="2.83695868220296E-05" />
-        </inertial> -->
+      </inertial>
       <visual>
         <origin xyz="0 0 0" rpy="0 0 0" />
@@ -76,9 +76,9 @@
   <xacro:macro name="inner_finger" params="prefix fingerprefix stroke">
     <link name="${prefix}${fingerprefix}_inner_finger">
-      <!--<inertial>
+      <inertial>
         <origin xyz="0.000299999999999317 0.0160078233491243 -0.0136945669206257" rpy="0 0 0" />
         <mass value="0.0104003125914103" />
         <inertia ixx="2.71909453810972E-06" ixy="1.35402465472579E-21" ixz="-7.1817349065269E-22" iyy="7.69100314106116E-07" iyz="6.74715432769696E-07" izz="2.30315190420171E-06" />
-        </inertial> -->
+      </inertial>
       <visual>
         <origin xyz="0 0 0" rpy="0 0 0" />

File: robotiq_2f_85_gripper_visualization/urdf/robotiq_arg2f_transmission.xacro (robot description, xacro)
@@ -11,4 +11,37 @@
       </actuator>
     </transmission>
+    <gazebo>
+         <!-- loading plugin: mimic joints works in gazebo now-->
+         <plugin filename="libroboticsgroup_upatras_gazebo_mimic_joint_plugin.so" name="${prefix}mimic_robotiq_85_4">
+            <joint>${prefix}finger_joint</joint>
+            <mimicJoint>${prefix}right_outer_knuckle_joint</mimicJoint>
+            <!--<multiplier>-1.0</multiplier>-->
+            <!--<offset>0.0</offset>-->
+        </plugin>
+        <plugin filename="libroboticsgroup_upatras_gazebo_mimic_joint_plugin.so" name="${prefix}mimic_robotiq_85_2">
+            <joint>${prefix}finger_joint</joint>
+            <mimicJoint>${prefix}left_inner_finger_joint</mimicJoint>
+            <!--<multiplier>1.0</multiplier>-->
+            <!--<offset>0.0</offset>-->
+        </plugin>
+        <plugin filename="libroboticsgroup_upatras_gazebo_mimic_joint_plugin.so" name="${prefix}mimic_robotiq_85_1">
+            <joint>${prefix}finger_joint</joint>
+            <mimicJoint>${prefix}right_inner_finger_joint</mimicJoint>
+            <!--<multiplier>1.0</multiplier>-->
+            <!--<offset>0.0</offset>-->
+        </plugin>
+        <plugin filename="libroboticsgroup_upatras_gazebo_mimic_joint_plugin.so" name="${prefix}mimic_robotiq_85_3">
+            <joint>${prefix}finger_joint</joint>
+            <mimicJoint>${prefix}left_inner_knuckle_joint</mimicJoint>
+            <!--<multiplier>-1.0</multiplier>-->
+            <!--<offset>0.0</offset>-->
+        </plugin>
+        <plugin filename="libroboticsgroup_upatras_gazebo_mimic_joint_plugin.so" name="${prefix}mimic_robotiq_85_5">
+            <joint>${prefix}finger_joint</joint>
+            <mimicJoint>${prefix}right_inner_knuckle_joint</mimicJoint>
+            <!--<multiplier>-1.0</multiplier>-->
+            <!--<offset>0.0</offset>-->
+        </plugin>
+    </gazebo>
   </xacro:macro>
 </robot>
